File: demo.sch (KiCad schematic (older format))
At the start: 24 parts, among them U1 STM32F103C8Tx

Commit message: update
Parts:
- added C?: 20pF, symbol Device:C
- added J?: USB_B_Micro, symbol Connector:USB_B_Micro
- added J?: Conn_01x06_Shielded, symbol Connector_Generic_Shielded:Conn_01x06_Shielded
- added Q?: S9013, Package_TO_SOT_THT:TO-92_Inline, symbol Transistor_BJT:S8050
- added R?: 100K, symbol Device:R
- added R? (x2): 100, symbol Device:R
- added R?: 36K, symbol Device:R
- added R?: 10K, symbol Device:R
- added R?: 1K5, symbol Device:R
- added U?: USBLC6-2SC6, Package_TO_SOT_SMD:SOT-23-6, symbol Power_Protection:USBLC6-2SC6
Connections:
- net +3V3: now also J?.1 (Pin_1), Q?.3 (C)
- net +5V: now also J?.1 (VBUS), R?.2, U?.5 (VBUS)
- net GND: now also C?.1, J?.5 (GND), J?.6 (Pin_6), J?.6 (Shield), J?.SH (Shield), R?.1, R?.1, U?.2 (GND)
- net NRST: now also J?.4 (Pin_4)
- net at U1.29 (PA8): now also R?.2
- net SWO: now reaches U1.31 (PA10)
- net SWO: now also J?.5 (Pin_5)
- net STLINK_USB_DM: now reaches U1.32 (PA11)
- net STLINK_USB_DM: now also J?.3 (D+), U?.1 (IO1), U?.6 (IO1)
- net STLINK_USB_DP: now reaches U1.33 (PA12)
- net STLINK_USB_DP: now also J?.2 (D-), R?.1, U?.3 (IO2), U?.4 (IO2)
- net STM_JTMS: now reaches U1.34 (PA13)
- net STM_JTCK: now reaches U1.37 (PA14)
- net USB_RENUMn: now reaches U1.38 (PA15)
- net USB_RENUMn: now also R?.1
- new net: J?.4 (ID), R?.2
- new net: Q?.1 (E), R?.2
- new net: Q?.2 (B), R?.1, R?.2, R?.2
- new net: C?.2, R?.1
- new net SWCLK: J?.3 (Pin_3)
- new net SWDIO: J?.2 (Pin_2)
Other:
- note added: "COM\n"
- note added: "Interface"
- note added: "MCU"
- note added: "USB"
- note added: "filter cap\n"
- note added: "power convert"

Commit message: update pcb and sch
Parts:
- removed C?: 20pF, symbol Device:C
- removed J?: Conn_01x06_Shielded, symbol Connector_Generic_Shielded:Conn_01x06_Shielded
- removed Q?: S9013, Package_TO_SOT_THT:TO-92_Inline, symbol Transistor_BJT:S8050
- removed R? (x3): 10K, symbol Device:R
- removed R? (x2): 100, symbol Device:R
- removed R?: 36K, symbol Device:R
- removed R?: 1K5, symbol Device:R
- removed U?: AMS1117CS-3.3, Package_SO:SOIC-8_3.9x4.9mm_P1.27mm, symbol Regulator_Linear:AMS1117CS-3.3
- removed U?: USBLC6-2SC6, Package_TO_SOT_SMD:SOT-23-6, symbol Power_Protection:USBLC6-2SC6
- added J1: download_firmware, hardware-demo:PinHeader_1x04_P2.54mm_Vertical, symbol Connector_Generic:Conn_01x04
- added J3: stlink_interface, hardware-demo:PinHeader_1x06_P2.54mm_Horizontal, symbol Connector_Generic:Conn_01x06
- added R4, R5, R6, R7: 22, hardware-demo:R_0603_1608Metric, symbol Device:R
- added R9: 100R, hardware-demo:R_0603_1608Metric, symbol Device:R
- added U2: AMS1117-3.3, hardware-demo:SOT-223-3_TabPin2, symbol Regulator_Linear:AMS1117-3.3
- C1, C7: renamed from C?; footprint (none) -> hardware-demo:C_0805_2012Metric_Pad1.15x1.40mm_HandSolder
- C10, C11, C2, C3, C4, C5, C6, C8, C9: renamed from C?; footprint (none) -> hardware-demo:C_0603_1608Metric
- D1, D2: renamed from D?; footprint (none) -> hardware-demo:LED_0603_1608Metric
- J2: renamed from J?; footprint (none) -> hardware-demo:USB_Micro-B_Amphenol_10103594-0001LF_Horizontal
- R1, R12, R13, R14, R2, R3, R8: renamed from R?; footprint (none) -> hardware-demo:R_0603_1608Metric
- U1: footprint Package_QFP:LQFP-48_7x7mm_P0.5mm -> hardware-demo:LQFP-48_7x7mm_P0.5mm
- Y1: renamed from Y?; footprint (none) -> hardware-demo:Crystal_SMD_3215-2Pin_3.2x1.5mm
Connections:
- net +3V3: now also J1.1 (Pin_1), J3.1 (Pin_1), U2.2 (VO)
- net +5V: now also U2.3 (VI)
- net GND: now also J1.4 (Pin_4), J3.6 (Pin_6), U2.1 (GND)
- net STLINK_USB_DM: now also J2.2 (D-); no longer J2.3 (D+)
- net STLINK_USB_DP: now also J2.3 (D+); no longer J2.2 (D-)
- net STM_JTCK: now also J1.3 (Pin_3)
- net STM_JTMS: now also J1.2 (Pin_2)
- net SWCLK: now also J3.3 (Pin_3), R5.2
- net SWDIO: now also J3.2 (Pin_2), R4.2
- net SWO: now also R7.1
- net T_JTCK: now reaches U1.15 (PA5)
- net T_JTCK: now also U1.26 (PB13), R5.1
- net T_NRST: now reaches U1.18 (PB0)
- net T_NRST: now also R6.1
- net T_SWDIO_IN: now reaches U1.25 (PB12)
- net T_SWDIO_IN: now also R9.1
- net T_JTMS: now reaches U1.27 (PB14)
- net T_JTMS: now also R4.1, R9.2
- net USB_RENUMn: no longer names the net of U1.38 (PA15)
- new net: J3.4 (Pin_4), R6.2
- new net: J3.5 (Pin_5), R7.2
- no-connect marks 12 -> 16

Commit message: update pcb and sch
Connections:
- net STLINK_USB_DM renamed STLINK_USB_DM-
- net STLINK_USB_DP renamed STLINK_USB_DP+
Changed lines of the file:
@@
 T_NRST
 Text Label 3900 5050 0    50   ~ 0
-STLINK_USB_DP
+STLINK_USB_DP+
 Text Label 3700 5150 0    50   ~ 0
-STLINK_USB_DM
+STLINK_USB_DM-
 Wire Wire Line
 	8350 4350 9250 4350
@@
 	8350 4250 9250 4250
 Text Label 9250 4250 0    50   ~ 0
-STLINK_USB_DM
+STLINK_USB_DM-
 Text Label 9250 4350 0    50   ~ 0
-STLINK_USB_DP
+STLINK_USB_DP+
 Wire Wire Line
 	8350 4150 8950 4150

Commit message: v1.0.0
Parts:
- removed C2, C8: 0.1uF, hardware-demo:C_0603_1608Metric, symbol Device:C
- removed C7: 10uF, hardware-demo:C_0805_2012Metric_Pad1.15x1.40mm_HandSolder, symbol Device:C
- removed J2: USB_B_Micro, hardware-demo:USB_Micro-B_Amphenol_10103594-0001LF_Horizontal, symbol Connector:USB_B_Micro
- removed U2: AMS1117-3.3, hardware-demo:SOT-223-3_TabPin2, symbol Regulator_Linear:AMS1117-3.3
- added C2, C3: 10uF, Capacitor_Tantalum_SMD:CP_EIA-1608-10_AVX-L, symbol Device:CP
- added C4: 0.1uF, hardware-demo:C_0402_1005Metric, symbol Device:C
- added J1: USB_C_Receptacle_USB2.0, hardware-demo:USB_C_Receptacle_Amphenol_12401610E4-2A, symbol Connector:USB_C_Receptacle_USB2.0
- added U1: XC6220B331MR, hardware-demo:SOT-23-5, symbol Regulator_Linear:XC6220B331MR
- C1: value 10uF -> 0.1uF; footprint hardware-demo:C_0805_2012Metric_Pad1.15x1.40mm_HandSolder -> hardware-demo:C_0402_1005Metric
- C10: renamed from C5; footprint hardware-demo:C_0603_1608Metric -> hardware-demo:C_0402_1005Metric
- C11: renamed from C6; footprint hardware-demo:C_0603_1608Metric -> hardware-demo:C_0402_1005Metric
- C5: renamed from C11; footprint hardware-demo:C_0603_1608Metric -> hardware-demo:C_0402_1005Metric
- C6: renamed from C9; footprint hardware-demo:C_0603_1608Metric -> hardware-demo:C_0402_1005Metric
- C7: renamed from C10; footprint hardware-demo:C_0603_1608Metric -> hardware-demo:C_0402_1005Metric
- C8: renamed from C3; footprint hardware-demo:C_0603_1608Metric -> hardware-demo:C_0402_1005Metric
- C9: renamed from C4; footprint hardware-demo:C_0603_1608Metric -> hardware-demo:C_0402_1005Metric
- D1, D2: footprint hardware-demo:LED_0603_1608Metric -> hardware-demo:LED_0402_1005Metric
- J2: renamed from J1; footprint hardware-demo:PinHeader_1x04_P2.54mm_Vertical -> Connector_PinHeader_1.27mm:PinHeader_1x04_P1.27mm_Vertical
- J3: footprint hardware-demo:PinHeader_1x06_P2.54mm_Horizontal -> hardware-demo:PinHeader_1x06_P1.27mm_Horizontal
- R1: renamed from R8; footprint hardware-demo:R_0603_1608Metric -> hardware-demo:R_0402_1005Metric
- R10: renamed from R4; footprint hardware-demo:R_0603_1608Metric -> hardware-demo:R_0402_1005Metric
- R11: renamed from R6; footprint hardware-demo:R_0603_1608Metric -> hardware-demo:R_0402_1005Metric
- R12: renamed from R7; footprint hardware-demo:R_0603_1608Metric -> hardware-demo:R_0402_1005Metric
- R2: renamed from R12; footprint hardware-demo:R_0603_1608Metric -> hardware-demo:R_0402_1005Metric
- R3: renamed from R1; footprint hardware-demo:R_0603_1608Metric -> hardware-demo:R_0402_1005Metric
- R4: renamed from R2; footprint hardware-demo:R_0603_1608Metric -> hardware-demo:R_0402_1005Metric
- R5: renamed from R13; footprint hardware-demo:R_0603_1608Metric -> hardware-demo:R_0402_1005Metric
- R6: renamed from R14; footprint hardware-demo:R_0603_1608Metric -> hardware-demo:R_0402_1005Metric
- R7: renamed from R9; footprint hardware-demo:R_0603_1608Metric -> hardware-demo:R_0402_1005Metric
- R8: renamed from R3; value 100K -> 5K1; footprint hardware-demo:R_0603_1608Metric -> hardware-demo:R_0402_1005Metric
- R9: renamed from R5; footprint hardware-demo:R_0603_1608Metric -> hardware-demo:R_0402_1005Metric
- renumbered U1 to U2
Connections:
- net +3V3: now also C3.1, C4.1, U1.5 (VOUT)
- net +5V: now also C2.1, J1.A4 (VBUS), J1.A9 (VBUS), J1.B4 (VBUS), J1.B9 (VBUS), U1.1 (VIN), U1.3 (CE)
- net GND: now also J3.4 (Pin_4), C2.2, C3.2, C4.2, J1.A1 (GND), J1.A12 (GND), J1.B1 (GND), J1.B12 (GND), J1.S1 (SHIELD), U1.2 (GND); no longer J3.6 (Pin_6)
- net STLINK_USB_DM-: now also J1.A7 (D-), J1.B7 (D-)
- net STLINK_USB_DP+: now also J1.A6 (D+), J1.B6 (D+)
- net SWCLK: now also J3.2 (Pin_2); no longer J3.3 (Pin_3)
- net SWDIO: now also J3.3 (Pin_3); no longer J3.2 (Pin_2)
- net at R8.2: now also J1.A5 (CC1), J1.B5 (CC2)
- net at R11.2: now also J3.5 (Pin_5); no longer J3.4 (Pin_4)
- net at R12.2: now also J3.6 (Pin_6); no longer J3.5 (Pin_5)
- no-connect marks 16 -> 24
Other:
- moved on the sheet: R10, R11, R12, R8, R9
