File: demo.kicad_pcb (KiCad board)
At the start: 4 copper layers, 36 x 12.5 mm, 32 parts, among them J2 Conn_01x06, J3 Conn_01x04, J4 USB_C_Receptacle, U1 Regulator_Linear_XC6220B331MR, U2 MCU_ST_STM32F1_STM32F103C8Tx, Y2 8M

Commit message: update files
Parts:
- moved C5 17.0 mm to (118.6, 110.9), turned to 0 degrees
- moved C3 11.0 mm to (118.7, 101.5), turned to 180 degrees
- moved R8 9.18 mm to (124.8, 104.6), turned to 0 degrees
- moved C7 7.30 mm to (125.0, 110.3)
- moved C8 6.90 mm to (123.4, 111.4), turned to 180 degrees
- moved C10 6.42 mm to (106.5, 102.3), turned to 180 degrees
- moved C4 6.13 mm to (110.2, 110.9), turned to 180 degrees
- moved R4 6.13 mm to (103.8, 106.3), turned to 180 degrees
- moved C9 6.10 mm to (106.5, 107.4), turned to 0 degrees
- moved Y2 6.08 mm to (107.3, 104.8)
- moved R11 6.06 mm to (103.8, 108.7)
- moved R5 5.89 mm to (103.8, 105.0), turned to 180 degrees
- moved R6 5.72 mm to (103.8, 103.8), turned to 180 degrees
- moved U2 5.67 mm to (114.4, 106.2)
- moved R7 5.63 mm to (103.8, 102.6), turned to 180 degrees
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Routing:
- net GND: track 24.8 -> 9.06 mm, vias 21 -> 2
- net Net-(J4-CC1): track 11.0 -> 16.5 mm, vias 3 -> 5
- net +3V3: track 18.7 -> 23.5 mm, vias 17 -> 15
- net /BOOT0: track 7.01 -> 11.7 mm, vias 0 -> 2
- net Net-(U2-PA0): track 3.30 -> 7.97 mm, vias 0 -> 2
- net /T_NRST: track 13.1 -> 16.4 mm
- net /T_JTMS: track 20.1 -> 16.9 mm
- net /T_JTCK: track 16.7 -> 19.2 mm, vias 2 -> 3
- net /STLINK_USB_DM-: track 15.6 -> 13.3 mm, vias 2 -> 3
- net /LED_STLINK: track 6.37 -> 4.49 mm, vias 2 -> 0
- net /STLINK_USB_DP+: track 13.1 -> 11.5 mm
- net /SWO: track 18.0 -> 16.5 mm
- net Net-(U2-PD1): track 5.13 -> 4.08 mm
- net /SWCLK: track 1.69 -> 2.56 mm
- net /SWDIO: track 1.75 -> 2.51 mm
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Other:
- board size 36 x 12.5 mm -> 35 x 12.5 mm
- board text added: "3V3"
- board text added: "GND"
- board text added: "NRST"
- board text added: "SWCLK"
- board text added: "SWDIO"
- board text added: "SWO"
- board text added: "Type-C STLINK"

Commit message: update
Routing:
- net +3V3: track 23.5 -> 27.1 mm
Changed lines of the file:
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@@
       (dashed_line_gap_ratio 3.000000)
       (svgprecision 4)
-      (plotframeref false)
+      (plotframeref true)
       (viasonmask false)
       (mode 1)
-      (useauxorigin false)
+      (useauxorigin true)
       (hpglpennumber 1)
       (hpglpenspeed 20)
@@
       (plotvalue true)
       (plotinvisibletext false)
-      (sketchpadsonfab false)
+      (sketchpadsonfab true)
       (subtractmaskfromsilk false)
       (outputformat 1)
@@
     (effects (font (size 0.8128 0.8128) (thickness 0.1524) bold) (justify left bottom mirror))
   )
-  (gr_text "Type-C STLINK" (at 117.094 101.854 90) (layer "B.SilkS")
+  (gr_text "Type-C STLINK" (at 107.2 110.8 -90) (layer "B.SilkS")
     (effects (font (size 0.8128 0.8128) (thickness 0.1524) bold) (justify left bottom mirror))
   )
@@
   (segment (start 118.16 110.88) (end 118.16 110.890438) (width 0.254) (layer "F.Cu") (net 3))
   (segment (start 119.269562 112) (end 120.5 112) (width 0.254) (layer "F.Cu") (net 3))
+  (segment (start 121.7 112) (end 120.5 112) (width 0.254) (layer "F.Cu") (net 3))
   (segment (start 123.84 111.355) (end 124.755 111.355) (width 0.254) (layer "F.Cu") (net 3))
   (segment (start 123.52 109.9725) (end 123.8825 109.9725) (width 0.254) (layer "F.Cu") (net 3))
@@
   (segment (start 111.68 102.0175) (end 111.68 103.06) (width 0.254) (layer "F.Cu") (net 3))
   (segment (start 117.7175 110.88) (end 117.18 110.3425) (width 0.254) (layer "F.Cu") (net 3))
+  (segment (start 123.84 111.365438) (end 123.205438 112) (width 0.254) (layer "F.Cu") (net 3))
   (segment (start 111.31 103.43) (end 110.2675 103.43) (width 0.254) (layer "F.Cu") (net 3))
   (segment (start 123.4 104.59) (end 124.3 104.59) (width 0.254) (layer "F.Cu") (net 3))
   (segment (start 111.073514 107.43) (end 110.2675 107.43) (width 0.254) (layer "F.Cu") (net 3))
+  (segment (start 123.205438 112) (end 121.7 112) (width 0.254) (layer "F.Cu") (net 3))
   (segment (start 120.71 101.49) (end 120.78 101.56) (width 0.254) (layer "F.Cu") (net 3))
   (segment (start 110.68 110.036486) (end 111.332 109.384486) (width 0.254) (layer "F.Cu") (net 3))
   (segment (start 110.65 101.49) (end 111.1525 101.49) (width 0.254) (layer "F.Cu") (net 3))
+  (segment (start 123.84 111.355) (end 123.84 111.365438) (width 0.254) (layer "F.Cu") (net 3))
   (segment (start 101.72 109.42) (end 102.215 109.915) (width 0.254) (layer "F.Cu") (net 3))
   (segment (start 119.14 101.49) (end 119.14 102.8825) (width 0.254) (layer "F.Cu") (net 3))
@@
   (segment (start 122.34 100.58) (end 117.18 100.58) (width 0.1) (layer "B.Cu") (net 14))
   (segment (start 123.32 101.56) (end 122.34 100.58) (width 0.1) (layer "B.Cu") (net 14))
-  (segment (start 130.25 103.6) (end 130 103.6) (width 0.1) (layer "F.Cu") (net 17))
   (segment (start 125.31 103.6) (end 126.01 103.6) (width 0.1) (layer "F.Cu") (net 17))
-  (segment (start 130.96 104.31) (end 130.25 103.6) (width 0.1) (layer "F.Cu") (net 17))
+  (segment (start 130.96 104.56) (end 130 103.6) (width 0.1) (layer "F.Cu") (net 17))
+  (segment (start 129.62 105.92) (end 129.32 105.62) (width 0.1) (layer "F.Cu") (net 17))
+  (segment (start 127.115 106.87) (end 126.12 106.87) (width 0.1) (layer "F.Cu") (net 17))
   (segment (start 129.62 106.86) (end 129.62 105.92) (width 0.1) (layer "F.Cu") (net 17))
-  (segment (start 130.96 106.53) (end 130.96 104.31) (width 0.1) (layer "F.Cu") (net 17))
-  (segment (start 127.115 106.87) (end 126.12 106.87) (width 0.1) (layer "F.Cu") (net 17))
-  (segment (start 129.32 105.62) (end 128.415 105.62) (width 0.1) (layer "F.Cu") (net 17))
-  (segment (start 129.62 105.92) (end 129.32 105.62) (width 0.1) (layer "F.Cu") (net 17))
-  (segment (start 128.44 105.595) (end 128.415 105.62) (width 0.1) (layer "F.Cu") (net 17))
   (segment (start 129.63 106.87) (end 129.62 106.86) (width 0.1) (layer "F.Cu") (net 17))
+  (segment (start 130.96 106.53) (end 130.96 104.56) (width 0.1) (layer "F.Cu") (net 17))
+  (segment (start 128.415 105.62) (end 129.32 105.62) (width 0.1) (layer "F.Cu") (net 17))
   (via micro (at 126.01 103.6) (size 0.25) (drill 0.15) (layers "F.Cu" "B.Cu") (net 17))
   (via micro (at 126.12 106.87) (size 0.25) (drill 0.15) (layers "F.Cu" "B.Cu") (net 17))
@@
   (segment (start 113.68 102.0175) (end 113.68 100.51) (width 0.1) (layer "F.Cu") (net 33))
   (segment (start 104.35 100.51) (end 104.35 101.36) (width 0.1) (layer "F.Cu") (net 33))
-  (via micro (at 104.35 100.51) (size 0.25) (drill 0.15) (layers "F.Cu" "B.Cu") (free) (net 33))
-  (via micro (at 113.68 100.51) (size 0.25) (drill 0.15) (layers "F.Cu" "B.Cu") (free) (net 33))
-  (segment (start 113.68 100.51) (end 104.35 100.51) (width 0.1) (layer "B.Cu") (net 33))
+  (via micro (at 104.35 100.58) (size 0.25) (drill 0.15) (layers "F.Cu" "B.Cu") (free) (net 33))
+  (via micro (at 113.68 100.58) (size 0.25) (drill 0.15) (layers "F.Cu" "B.Cu") (free) (net 33))
+  (segment (start 104.35 100.58) (end 113.68 100.58) (width 0.1) (layer "B.Cu") (net 33))
   (segment (start 120.06 108.93) (end 120.08 108.91) (width 0.1) (layer "F.Cu") (net 34))
   (segment (start 118.5925 108.93) (end 120.06 108.93) (width 0.1) (layer "F.Cu") (net 34))

Commit message: update to product
Routing:
- net +3V3: track 27.1 -> 28.5 mm, vias 15 -> 9
- net /BOOT0: track 11.7 -> 11.0 mm
- net Net-(J4-CC1): track 16.3 -> 16.8 mm
Other:
- board text added: "TypeC-STLINK-Fake"
- board text removed: "Type-C STLINK"

Commit message: update sch
Parts:
- removed C1, C11, C3, C4, C5, C6, C8: 100nF, Capacitor_SMD:C_0402_1005Metric
- removed C10, C9: 10pF, Capacitor_SMD:C_0402_1005Metric
- removed C2, C7: 10uF, Capacitor_SMD:C_0603_1608Metric
- removed D1, D2: LED, LED_SMD:LED_0402_1005Metric
- removed J2: Conn_01x06, Connector_PinHeader_1.27mm:PinHeader_1x06_P1.27mm_Horizontal
- removed J3: Conn_01x04, Connector_PinHeader_1.27mm:PinHeader_1x04_P1.27mm_Vertical
- removed J4: USB_C_Receptacle, selfdefined_library:USB_C_Receptacle_24Pin_Hole_SMD
- removed R1, R10, R2: 100, Resistor_SMD:R_0402_1005Metric
- removed R11, R3, R9: 100K, Resistor_SMD:R_0402_1005Metric
- removed R12, R13: 4K7, Resistor_SMD:R_0402_1005Metric
- removed R4, R5, R6, R7: 22, Resistor_SMD:R_0402_1005Metric
- removed R8: 1.5K, Resistor_SMD:R_0402_1005Metric
- removed U1: Regulator_Linear_XC6220B331MR, Package_TO_SOT_SMD:SOT-23-5
- removed U2: MCU_ST_STM32F1_STM32F103C8Tx, Package_QFP:LQFP-48_7x7mm_P0.5mm
- removed Y2: 8M, Crystal:Crystal_SMD_3225-4Pin_3.2x2.5mm
Routing:
- net T_JTCK: track 0.00 -> 19.2 mm
- net /T_JTCK: track 19.2 -> 0.00 mm, vias 3 -> 0
- net T_NRST: track 0.00 -> 16.4 mm
- net /T_NRST: track 16.4 -> 0.00 mm, vias 2 -> 0
- net SWO: track 0.00 -> 16.2 mm
- net /SWO: track 16.2 -> 0.00 mm, vias 2 -> 0
- net STLINK_USB_DM-: track 0.00 -> 13.1 mm
- net /STLINK_USB_DM-: track 13.1 -> 0.00 mm, vias 3 -> 0
- net STLINK_USB_DP+: track 0.00 -> 11.6 mm
- net /STLINK_USB_DP+: track 11.6 -> 0.00 mm, vias 2 -> 0
- net STM_JTCK: track 0.00 -> 7.81 mm
- net /STM_JTCK: track 7.81 -> 0.00 mm, vias 1 -> 0
- net STM_JTMS: track 0.00 -> 5.83 mm
- net /STM_JTMS: track 5.83 -> 0.00 mm, vias 1 -> 0
- net LED_STLINK: track 0.00 -> 4.49 mm
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- removed copper zone on In2.Cu, net +3V3
- removed copper zone on In1.Cu, net GND
Other:
- board outline removed
- board text removed: "3V3"
- board text removed: "GND"
- board text removed: "NRST"
- board text removed: "SWCLK"
- board text removed: "SWDIO"
- board text removed: "SWO"
- board text removed: "TypeC-STLINK-Fake"
