File: demo.kicad_pcb (KiCad board)
At the start: 4 copper layers, 38 x 13 mm, 39 parts, among them J1 USB_C_Receptacle_USB2.0_16P, J2 Conn_02x05_Odd_Even, J3 Conn_01x04, Q1 S9013, U1 XC6206P332MR, U2 STM32F103CBT6, Y1 8M

Commit message: V1.0.4
Parts:
- J2: footprint Connector_PinHeader_2.54mm:PinHeader_2x05_P2.54mm_Horizontal -> Library:pin-header-hor-handsolid-2x5
- moved J2 5.22 mm to (117.1, 100.0)
Routing:
- net GND: track 30.5 -> 37.0 mm, vias 82 -> 61
- net Net-(J2-Pin_10): track 5.87 -> 3.13 mm, vias 0 -> 1
- net +3V3: track 20.6 -> 22.3 mm, vias 17 -> 18
- net Net-(J2-Pin_2): track 5.51 -> 3.88 mm, vias 0 -> 1
- net Net-(J2-Pin_6): track 6.81 -> 5.44 mm, vias 0 -> 1
- net /T_Tx: track 19.8 -> 18.6 mm, vias 2 -> 3
- net /T_Rx: track 19.8 -> 21.0 mm
- net Net-(J2-Pin_4): track 5.32 -> 4.15 mm, vias 0 -> 1
Other:
- board size 38 x 13 mm -> 34 x 13 mm
- board text added: "v1.0.4"
- board text removed: "v1.0.3"
